File: ESP8285-WLED.kicad_pcb (KiCad board)
At the start: 2 copper layers, 62.2 x 35.6 mm, 56 parts, among them J1 WLED, J2 USB_B_Micro, J3 ANT, Q1 UMH3N, SW1 RESET, SW2 FLASH, U1 ME3116, U2 ESP8285, U3 ME6211, U4 TXS0101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

Commit message: tweaking and cleanups
Parts:
- moved R7 11.9 mm to (126.0, 118.9), turned to 90 degrees
- moved R8 3.67 mm to (105.9, 110.2)
- moved C6 2.54 mm to (105.6, 106.3), turned to 0 degrees
- moved C7 1.84 mm to (105.6, 108.4), turned to 0 degrees
- moved J3 0.51 mm to (141.8, 118.4)
- moved C1 0.13 mm to (127.8, 118.9), turned to 90 degrees
Routing:
- net /CUTXD: track 4.18 -> 17.2 mm, vias 0 -> 2
- net /UTXD: track 18.2 -> 6.75 mm, vias 2 -> 0
- net /GPIO0: track 59.3 -> 55.4 mm
- net GND: track 11.2 -> 14.1 mm, vias 44 -> 48
- net +5V: track 44.0 -> 46.1 mm
- net /XO: track 10.9 -> 9.12 mm
- net Net-(R10-Pad2): track 21.8 -> 23.4 mm

Commit message: more tidying
Parts:
- moved R2 23.6 mm to (115.0, 121.3), turned to 180 degrees
- moved C13 1.84 mm to (137.9, 111.4)
- moved L2 1.59 mm to (137.9, 109.7)
Routing:
- net +3V3: track 103.7 -> 106.8 mm, vias 10 -> 9
- net /RST: track 41.1 -> 42.1 mm
- net GND: vias 48 -> 49

Commit message: adjustments around the crystal
Parts:
- moved R7 4.18 mm to (126.8, 114.8), turned to 0 degrees
- moved Y1 1.61 mm to (130.5, 117.4), turned to 315 degrees
- moved C2 1.56 mm to (132.7, 119.4), turned to 225 degrees
- moved C1 0.60 mm to (128.4, 118.9), turned to 135 degrees
- moved R1 0.51 mm to (136.3, 118.9)
Routing:
- net +3V3: track 106.8 -> 119.9 mm, vias 9 -> 11
- net /UTXD: track 6.75 -> 3.43 mm
- net /XO: track 9.12 -> 6.88 mm
- net /CUTXD: track 17.2 -> 19.1 mm
- net GND: track 14.1 -> 15.9 mm, vias 49 -> 51
- net /XI: track 7.65 -> 6.90 mm

Commit message: more tweaking
Parts:
- moved C12 14.7 mm to (135.1, 118.8), turned to 90 degrees
- moved R17 13.3 mm to (139.5, 102.6), turned to 270 degrees
- moved D4 9.68 mm to (139.5, 99.1), turned to 270 degrees
- moved C10 2.24 mm to (123.2, 105.2), turned to 270 degrees
- moved C14 1.52 mm to (125.1, 104.9), turned to 270 degrees
- moved R1 0.38 mm to (136.7, 118.9)
Routing:
- net +3V3: track 119.9 -> 130.9 mm, vias 11 -> 9
- net /GPIO2: track 9.04 -> 16.6 mm
- net /GPIO0: track 55.2 -> 49.5 mm
- net GND: track 15.9 -> 16.8 mm, vias 51 -> 54
- net /RST: track 42.2 -> 42.7 mm
